Commit message: this is new code for ROS2 humble with lots of improvements to the rover description, controllers, and navigation stack. The commit includes changes to the URDF files, launch files, controller configurations, and EKF configuration for better state estimation. The joy teleop configuration has also been updated for improved control.

File: src/rover_description/urdf/aries_gazebo.xacro (robot description, xacro)
@@ -4,5 +4,9 @@
   <!-- Gazebo Materials -->
   <gazebo reference="base_link">
-    <material>Gazebo/Gray</material>
+    <material>
+      <ambient>0.7 0.7 0.7 1</ambient>
+      <diffuse>0.7 0.7 0.7 1</diffuse>
+      <specular>0.1 0.1 0.1 1</specular>
+    </material>
     <mu1>0.2</mu1>
     <mu2>0.2</mu2>
@@ -45,7 +49,11 @@
   </gazebo>
   <gazebo reference="L_1_Wheel_Link">
-    <material>Gazebo/Black</material>
-    <mu1>1.0</mu1>
-    <mu2>1.0</mu2>
+    <material>
+      <ambient>0.05 0.05 0.05 1</ambient>
+      <diffuse>0.05 0.05 0.05 1</diffuse>
+      <specular>0.01 0.01 0.01 1</specular>
+    </material>
+    <mu1>2.0</mu1>
+    <mu2>2.0</mu2>
     <kp>1000000.0</kp>
     <kd>100.0</kd>
@@ -55,7 +63,11 @@
   </gazebo>
   <gazebo reference="L_2_Wheel_Link">
-    <material>Gazebo/Black</material>
-    <mu1>1.0</mu1>
-    <mu2>1.0</mu2>
+    <material>
+      <ambient>0.05 0.05 0.05 1</ambient>
+      <diffuse>0.05 0.05 0.05 1</diffuse>
+      <specular>0.01 0.01 0.01 1</specular>
+    </material>
+    <mu1>2.0</mu1>
+    <mu2>2.0</mu2>
     <kp>1000000.0</kp>
     <kd>100.0</kd>
@@ -65,7 +77,11 @@
   </gazebo>
   <gazebo reference="L_3_Wheel_Link">
-    <material>Gazebo/Black</material>
-    <mu1>1.0</mu1>
-    <mu2>1.0</mu2>
+    <material>
+      <ambient>0.05 0.05 0.05 1</ambient>
+      <diffuse>0.05 0.05 0.05 1</diffuse>
+      <specular>0.01 0.01 0.01 1</specular>
+    </material>
+    <mu1>2.0</mu1>
+    <mu2>2.0</mu2>
     <kp>1000000.0</kp>
     <kd>100.0</kd>
@@ -75,7 +91,11 @@
   </gazebo>
   <gazebo reference="R_1_Wheel_Link">
-    <material>Gazebo/Black</material>
-    <mu1>1.0</mu1>
-    <mu2>1.0</mu2>
+    <material>
+      <ambient>0.05 0.05 0.05 1</ambient>
+      <diffuse>0.05 0.05 0.05 1</diffuse>
+      <specular>0.01 0.01 0.01 1</specular>
+    </material>
+    <mu1>2.0</mu1>
+    <mu2>2.0</mu2>
     <kp>1000000.0</kp>
     <kd>100.0</kd>
@@ -85,7 +105,11 @@
   </gazebo>
   <gazebo reference="R_2_Wheel_Link">
-    <material>Gazebo/Black</material>
-    <mu1>1.0</mu1>
-    <mu2>1.0</mu2>
+    <material>
+      <ambient>0.05 0.05 0.05 1</ambient>
+      <diffuse>0.05 0.05 0.05 1</diffuse>
+      <specular>0.01 0.01 0.01 1</specular>
+    </material>
+    <mu1>2.0</mu1>
+    <mu2>2.0</mu2>
     <kp>1000000.0</kp>
     <kd>100.0</kd>
@@ -95,7 +119,11 @@
   </gazebo>
   <gazebo reference="R_3_Wheel_Link">
-    <material>Gazebo/Black</material>
-    <mu1>1.0</mu1>
-    <mu2>1.0</mu2>
+    <material>
+      <ambient>0.05 0.05 0.05 1</ambient>
+      <diffuse>0.05 0.05 0.05 1</diffuse>
+      <specular>0.01 0.01 0.01 1</specular>
+    </material>
+    <mu1>2.0</mu1>
+    <mu2>2.0</mu2>
     <kp>1000000.0</kp>
     <kd>100.0</kd>
@@ -242,5 +270,5 @@
       <use_pose_vector_msg>true</use_pose_vector_msg>
       <static_publisher>true</static_publisher>
-      <static_update_frequency>60</static_update_frequency>
+      <static_update_frequency>100</static_update_frequency>
     </plugin>
   </gazebo>
@@ -254,5 +282,5 @@
             <!-- <tf_topic>/model/aries/tf</tf_topic> -->
             <dimensions>2</dimensions>
-            <odom_publish_frequency>60</odom_publish_frequency>
+            <odom_publish_frequency>100</odom_publish_frequency>
         </plugin>
   </gazebo>
@@ -260,5 +288,5 @@
       <sensor name="imu_sensor" type="imu">
           <always_on>1</always_on>
-          <update_rate>60</update_rate>
+          <update_rate>100</update_rate>
           <gz_frame_id>imu_frame</gz_frame_id>
           <visualize>true</visualize>
@@ -284,11 +312,3 @@
     </gazebo>
   </xacro:unless>
-  <!-- gz_ros2_control: creates controller_manager inside Gazebo when use_sim=true -->
-  <xacro:if value="$(arg use_sim)">
-    <gazebo>
-      <plugin filename="gz_ros2_control-system" name="gz_ros2_control::GazeboSimROS2ControlPlugin">
-        <parameters>$(find rover_controllers)/config/diff_controller.yaml</parameters>
-      </plugin>
-    </gazebo>
-  </xacro:if>
 </robot>

File: src/rover_description/urdf/left_link.xacro (robot description, xacro)
@@ -38,5 +38,5 @@
     </joint>
     <!-- Left Wheel 1 -->
-    <link name="L_1_Wheel_Link">
+    <link name="L_3_Wheel_Link">
         <inertial>
             <origin xyz="0 0 0.0350608778434713" rpy="0 0 0"/>
@@ -53,5 +53,5 @@
             <origin xyz="0 0 0" rpy="0 0 0"/>
             <geometry>
-                <mesh filename="${mesh_location}/L_1_Wheel_Link.STL"/>
+                <mesh filename="${mesh_location}/L_3_Wheel_Link.STL"/>
             </geometry>
             <material name="blue"/>
@@ -65,8 +65,8 @@
     </link>
     <!-- Left Wheel 1 Joint -->
-    <joint name="L_1_Wheel_Joint" type="continuous">
+    <joint name="L_3_Wheel_Joint" type="continuous">
         <origin xyz="0.14142135623731 0.141421356237309 -0.08667" rpy="0 0 0"/>
         <parent link="L_Boggie_Link"/>
-        <child link="L_1_Wheel_Link"/>
+        <child link="L_3_Wheel_Link"/>
         <axis xyz="0 0 -1"/>
         <dynamics damping="0.01" friction="0.01"/>
@@ -108,5 +108,5 @@
     </joint>
     <!-- Left Wheel 3 -->
-    <link name="L_3_Wheel_Link">
+    <link name="L_1_Wheel_Link">
         <inertial>
             <origin xyz="0 0 0.0350608778434703" rpy="0 0 0"/>
@@ -123,5 +123,5 @@
             <origin xyz="0 0 0" rpy="0 0 0"/>
             <geometry>
-                <mesh filename="${mesh_location}/L_3_Wheel_Link.STL"/>
+                <mesh filename="${mesh_location}/L_1_Wheel_Link.STL"/>
             </geometry>
             <material name="blue"/>
@@ -135,8 +135,8 @@
     </link>
     <!-- Left Wheel 3 Joint -->
-    <joint name="L_3_Wheel_Joint" type="continuous">
+    <joint name="L_1_Wheel_Joint" type="continuous">
         <origin xyz="-0.261 0.1785 -0.0759999999999989" rpy="0 0 0"/>
         <parent link="L_Rocker_Link"/>
-        <child link="L_3_Wheel_Link"/>
+        <child link="L_1_Wheel_Link"/>
         <axis xyz="0 0 -1"/>
         <dynamics damping="0.01" friction="0.01"/>

File: src/rover_description/urdf/my_robot.urdf.xacro (robot description, xacro)
@@ -6,4 +6,7 @@
     <!-- <xacro:arg name="serial_port" default="/dev/ttyACM0" /> -->
     <!-- <xacro:property name="serial_port" value="$(arg serial_port)" /> -->
+    <!-- Flip right wheel joint axes for RViz display only; pass invert_right_wheels:=true
+         in the display description and leave it false for the hardware description. -->
+    <xacro:arg name="invert_right_wheels" default="false"/>
     <xacro:include filename="common_properties.xacro" />
     <xacro:include filename="aries_gazebo.xacro" />

File: src/rover_description/urdf/right_link.xacro (robot description, xacro)
@@ -41,5 +41,5 @@
     </joint>
     <!-- Right Wheel 1 -->
-    <link name="R_1_Wheel_Link">
+    <link name="R_3_Wheel_Link">
         <inertial>
             <origin xyz="0 0 0.0350608778434713" rpy="0 0 0"/>
@@ -56,5 +56,5 @@
             <origin xyz="0 0 0" rpy="0 0 0"/>
             <geometry>
-                <mesh filename="${mesh_location}/R_1_Wheel_Link.STL"/>
+                <mesh filename="${mesh_location}/R_3_Wheel_Link.STL"/>
             </geometry>
             <material name="blue"/>
@@ -68,9 +68,14 @@
     </link>
     <!-- Right Wheel 1 Joint -->
-    <joint name="R_1_Wheel_Joint" type="continuous">
+    <joint name="R_3_Wheel_Joint" type="continuous">
         <origin xyz="0.1542 -0.1266 -0.086" rpy="0 0 0"/>
         <parent link="R_Boggie_Link"/>
-        <child link="R_1_Wheel_Link"/>
-        <axis xyz="0 0 1"/>
+        <child link="R_3_Wheel_Link"/>
+        <xacro:if value="$(arg invert_right_wheels)">
+            <axis xyz="0 0 -1"/>
+        </xacro:if>
+        <xacro:unless value="$(arg invert_right_wheels)">
+            <axis xyz="0 0 1"/>
+        </xacro:unless>
         <dynamics damping="0.01" friction="0.01"/>
     </joint>
@@ -107,9 +112,14 @@
         <parent link="R_Boggie_Link"/>
         <child link="R_2_Wheel_Link"/>
-        <axis xyz="0 0 1"/>
+        <xacro:if value="$(arg invert_right_wheels)">
+            <axis xyz="0 0 -1"/>
+        </xacro:if>
+        <xacro:unless value="$(arg invert_right_wheels)">
+            <axis xyz="0 0 1"/>
+        </xacro:unless>
         <dynamics damping="0.01" friction="0.01"/>
     </joint>
     <!-- Right Wheel 3 -->
-    <link name="R_3_Wheel_Link">
+    <link name="R_1_Wheel_Link">
         <inertial>
             <origin xyz="0 0 0.0350608778434713" rpy="0 0 0"/>
@@ -126,5 +136,5 @@
             <origin xyz="0 0 0" rpy="0 0 0"/>
             <geometry>
-                <mesh filename="${mesh_location}/R_3_Wheel_Link.STL"/>
+                <mesh filename="${mesh_location}/R_1_Wheel_Link.STL"/>
             </geometry>
             <material name="blue"/>
@@ -138,9 +148,14 @@
     </link>
     <!-- Right Wheel 3 Joint -->
-    <joint name="R_3_Wheel_Joint" type="continuous">
+    <joint name="R_1_Wheel_Joint" type="continuous">
         <origin xyz="-0.276 -0.1541 -0.0760000000000001" rpy="0 0 0"/>
         <parent link="R_Rocker_Link"/>
-        <child link="R_3_Wheel_Link"/>
-        <axis xyz="0 0 1"/>
+        <child link="R_1_Wheel_Link"/>
+        <xacro:if value="$(arg invert_right_wheels)">
+            <axis xyz="0 0 -1"/>
+        </xacro:if>
+        <xacro:unless value="$(arg invert_right_wheels)">
+            <axis xyz="0 0 1"/>
+        </xacro:unless>
         <dynamics damping="0.01" friction="0.01"/>
     </joint>

File: src/rover_description/urdf/rover_control.xacro (robot description, xacro)
@@ -82,5 +82,7 @@
   </xacro:if>
   <!-- ================================================================
-       REAL HARDWARE  (ODrive via CAN bus)
+       REAL HARDWARE  (ODrive S1 x6 via CAN bus)
+       Velocity limits: ±11.52 rad/s (110 RPM rated, r=0.110 m → ~1.27 m/s)
+       Effort limits  : ±5 Nm (motor rated torque)
        ================================================================ -->
   <xacro:unless value="$(arg use_sim)">
@@ -90,14 +92,14 @@
         <param name="can">can0</param>
       </hardware>
-      <!-- LEFT WHEELS — node_id matches ODrive CAN node ID -->
+      <!-- LEFT WHEELS -->
       <joint name="L_1_Wheel_Joint">
-        <param name="node_id">0</param>
+        <param name="node_id">3</param>
         <command_interface name="velocity">
-          <param name="min">-18.85</param>  <!-- rad/s = 3.0 rev/s * 2pi -->
-          <param name="max">18.85</param>
+          <param name="min">-11.52</param>
+          <param name="max"> 11.52</param>
         </command_interface>
         <command_interface name="effort">
-          <param name="min">-10</param>    <!-- Nm -->
-          <param name="max">10</param>
+          <param name="min">-5</param>
+          <param name="max"> 5</param>
         </command_interface>
         <state_interface name="position"/>
@@ -106,12 +108,12 @@
       </joint>
       <joint name="L_2_Wheel_Joint">
-        <param name="node_id">2</param>
+        <param name="node_id">4</param>
         <command_interface name="velocity">
-          <param name="min">-200</param>
-          <param name="max">200</param>
+          <param name="min">-11.52</param>
+          <param name="max"> 11.52</param>
         </command_interface>
         <command_interface name="effort">
-          <param name="min">-10</param>
-          <param name="max">10</param>
+          <param name="min">-5</param>
+          <param name="max"> 5</param>
         </command_interface>
         <state_interface name="position"/>
@@ -120,12 +122,12 @@
       </joint>
       <joint name="L_3_Wheel_Joint">
-        <param name="node_id">4</param>
+        <param name="node_id">5</param>
         <command_interface name="velocity">
-          <param name="min">-200</param>
-          <param name="max">200</param>
+          <param name="min">-11.52</param>
+          <param name="max"> 11.52</param>
         </command_interface>
         <command_interface name="effort">
-          <param name="min">-10</param>
-          <param name="max">10</param>
+          <param name="min">-5</param>
+          <param name="max"> 5</param>
         </command_interface>
         <state_interface name="position"/>
@@ -135,12 +137,12 @@
       <!-- RIGHT WHEELS -->
       <joint name="R_1_Wheel_Joint">
-        <param name="node_id">1</param>
+        <param name="node_id">2</param>
         <command_interface name="velocity">
-          <param name="min">-200</param>
-          <param name="max">200</param>
+          <param name="min">-11.52</param>
+          <param name="max"> 11.52</param>
         </command_interface>
         <command_interface name="effort">
-          <param name="min">-10</param>
-          <param name="max">10</param>
+          <param name="min">-5</param>
+          <param name="max"> 5</param>
         </command_interface>
         <state_interface name="position"/>
@@ -149,12 +151,12 @@
       </joint>
       <joint name="R_2_Wheel_Joint">
-        <param name="node_id">3</param>
+        <param name="node_id">1</param>
         <command_interface name="velocity">
-          <param name="min">-200</param>
-          <param name="max">200</param>
+          <param name="min">-11.52</param>
+          <param name="max"> 11.52</param>
         </command_interface>
         <command_interface name="effort">
-          <param name="min">-10</param>
-          <param name="max">10</param>
+          <param name="min">-5</param>
+          <param name="max"> 5</param>
         </command_interface>
         <state_interface name="position"/>
@@ -163,12 +165,12 @@
       </joint>
       <joint name="R_3_Wheel_Joint">
-        <param name="node_id">5</param>
+        <param name="node_id">0</param>
         <command_interface name="velocity">
-          <param name="min">-200</param>
-          <param name="max">200</param>
+          <param name="min">-11.52</param>
+          <param name="max"> 11.52</param>
         </command_interface>
         <command_interface name="effort">
-          <param name="min">-10</param>
-          <param name="max">10</param>
+          <param name="min">-5</param>
+          <param name="max"> 5</param>
         </command_interface>
         <state_interface name="position"/>
