Commit message: Update rover_description: launch/urdf tweaks, IMU/trajectory scripts, drop keyboard teleop
- Replace teleop_keyboard.py with imu_restamp.py, imu_to_tf.py, trajectory.py, traje.launch.py
- Add empty_world.sdf, remove xbox.config.yaml
- Update launch files, xacro URDFs, gazebo bridge config, and rviz display config

Co-Authored-By: Claude Sonnet 5 <noreply@anthropic.com>

File: rover_description/urdf/aries_base.xacro (robot description, xacro)
@@ -36,10 +36,4 @@
         <child link="imu_frame"/>
         <origin xyz="0.0 0.0 0.08" rpy="0.0 0.0 0.0"/>
-    </joint>
-    <link name="odom"/>
-    <joint name="odom_joint" type="fixed">
-        <parent link="odom"/>
-        <child link="base_footprint"/>
-        <origin xyz="0.0 0.0 0.0" rpy="0.0 0.0 0.0"/>
     </joint>
     <!-- Base Footprint -->

File: rover_description/urdf/left_link.xacro (robot description, xacro)
@@ -37,8 +37,8 @@
         <dynamics damping="50" friction="50"/>
     </joint>
-    <!-- Left Wheel 1 -->
+    <!-- Left Wheel 3 -->
     <link name="L_3_Wheel_Link">
         <inertial>
-            <origin xyz="0 0 0.0350608778434713" rpy="0 0 0"/>
+            <origin xyz="0 -0.0350608778434713 0" rpy="1.57 0 0"/>
             <mass value="${wheel_mass}"/>
             <inertia
@@ -51,5 +51,5 @@
         </inertial>
         <visual>
-            <origin xyz="0 0 0" rpy="0 0 0"/>
+            <origin xyz="0 0 0" rpy="1.57 0 0"/>
             <geometry>
                 <mesh filename="${mesh_location}/L_3_Wheel_Link.STL"/>
@@ -58,5 +58,5 @@
         </visual>
         <collision>
-            <origin xyz="0 0 0.035" rpy="0 0 0"/>
+            <origin xyz="0 -0.035 0" rpy="1.57 0 0"/>
             <geometry>
                 <cylinder radius="${wheel_radius}" length="${wheel_thickness}"/>
@@ -64,10 +64,10 @@
         </collision>
     </link>
-    <!-- Left Wheel 1 Joint -->
+    <!-- Left Wheel 3 Joint -->
     <joint name="L_3_Wheel_Joint" type="continuous">
-        <origin xyz="0.14142135623731 0.141421356237309 -0.08667" rpy="0 0 0"/>
+        <origin xyz="0.14142135623731 0.141421356237309 -0.08667" rpy="1.57 -3.14 0"/>
         <parent link="L_Boggie_Link"/>
         <child link="L_3_Wheel_Link"/>
-        <axis xyz="0 0 -1"/>
+        <axis xyz="0 1 0"/>
         <dynamics damping="0.01" friction="0.01"/>
     </joint>
@@ -75,5 +75,5 @@
     <link name="L_2_Wheel_Link">
         <inertial>
-            <origin xyz="0 0 0.0350608778434713" rpy="0 0 0"/>
+            <origin xyz="0 -0.0350608778434713 0" rpy="1.57 0 0"/>
             <mass value="${wheel_mass}"/>
             <inertia
@@ -86,5 +86,5 @@
         </inertial>
         <visual>
-            <origin xyz="0 0 0" rpy="0 0 0"/>
+            <origin xyz="0 0 0" rpy="1.57 0 0"/>
             <geometry>
                 <mesh filename="${mesh_location}/L_2_Wheel_Link.STL"/>
@@ -93,5 +93,5 @@
         </visual>
         <collision>
-            <origin xyz="0 0 0.035" rpy="0 0 0"/>
+            <origin xyz="0 -0.035 0" rpy="1.57 0 0"/>
             <geometry>
                 <cylinder radius="${wheel_radius}" length="${wheel_thickness}"/>
@@ -101,14 +101,14 @@
     <!-- Left Wheel 2 Joint -->
     <joint name="L_2_Wheel_Joint" type="continuous">
-        <origin xyz="-0.141421356237308 0.141421356237311 -0.08667" rpy="0 0 0"/>
+        <origin xyz="-0.141421356237308 0.141421356237311 -0.08667" rpy="1.57 -3.14 0"/>
         <parent link="L_Boggie_Link"/>
         <child link="L_2_Wheel_Link"/>
-        <axis xyz="0 0 -1"/>
+        <axis xyz="0 1 0"/>
         <dynamics damping="0.01" friction="0.01"/>
     </joint>
-    <!-- Left Wheel 3 -->
+    <!-- Left Wheel 1 -->
     <link name="L_1_Wheel_Link">
         <inertial>
-            <origin xyz="0 0 0.0350608778434703" rpy="0 0 0"/>
+            <origin xyz="0 -0.0350608778434703 0" rpy="1.57 0 0"/>
             <mass value="${wheel_mass}"/>
             <inertia
@@ -121,5 +121,5 @@
         </inertial>
         <visual>
-            <origin xyz="0 0 0" rpy="0 0 0"/>
+            <origin xyz="0 0 0" rpy="1.57 0 0"/>
             <geometry>
                 <mesh filename="${mesh_location}/L_1_Wheel_Link.STL"/>
@@ -128,5 +128,5 @@
         </visual>
         <collision>
-            <origin xyz="0 0 0.035" rpy="0 0 0"/>
+            <origin xyz="0 -0.035 0" rpy="1.57 0 0"/>
             <geometry>
                 <cylinder radius="${wheel_radius}" length="${wheel_thickness}"/>
@@ -134,10 +134,10 @@
         </collision>
     </link>
-    <!-- Left Wheel 3 Joint -->
+    <!-- Left Wheel 1 Joint -->
     <joint name="L_1_Wheel_Joint" type="continuous">
-        <origin xyz="-0.261 0.1785 -0.0759999999999989" rpy="0 0 0"/>
+        <origin xyz="-0.261 0.1785 -0.0759999999999989" rpy="1.57 -3.14 0"/>
         <parent link="L_Rocker_Link"/>
         <child link="L_1_Wheel_Link"/>
-        <axis xyz="0 0 -1"/>
+        <axis xyz="0 1 0"/>
         <dynamics damping="0.01" friction="0.01"/>
     </joint>

File: rover_description/urdf/my_robot.urdf.xacro (robot description, xacro)
@@ -6,7 +6,4 @@
     <!-- <xacro:arg name="serial_port" default="/dev/ttyACM0" /> -->
     <!-- <xacro:property name="serial_port" value="$(arg serial_port)" /> -->
-    <!-- Flip right wheel joint axes for RViz display only; pass invert_right_wheels:=true
-         in the display description and leave it false for the hardware description. -->
-    <xacro:arg name="invert_right_wheels" default="false"/>
     <xacro:include filename="common_properties.xacro" />
     <xacro:include filename="aries_gazebo.xacro" />
@@ -16,9 +13,3 @@
     <xacro:include filename="right_link.xacro" />
     <xacro:include filename="rover_control.xacro" />
-    <!-- <xacro:include filename="lidar.xacro" /> -->
-    <!-- <xacro:include filename="camera.xacro" /> -->
-   <!-- <xacro:include filename="d435i.xacro" /> -->
-    <!-- <xacro:include filename="arm.xacro" /> -->
-    <!-- <xacro:include filename="igus_rebel_robot2.urdf.xacro" /> -->
-    <!-- <xacro:include filename="igus_rebel2.control.xacro" /> -->
 </robot>

File: rover_description/urdf/right_link.xacro (robot description, xacro)
@@ -40,8 +40,8 @@
         <dynamics damping="50" friction="50"/>
     </joint>
-    <!-- Right Wheel 1 -->
+    <!-- Right Wheel 3 -->
     <link name="R_3_Wheel_Link">
         <inertial>
-            <origin xyz="0 0 0.0350608778434713" rpy="0 0 0"/>
+            <origin xyz="0 0.0350608778434713 0" rpy="-1.57 0 0"/>
             <mass value="${wheel_mass}"/>
             <inertia
@@ -54,5 +54,5 @@
             </inertial>
         <visual>
-            <origin xyz="0 0 0" rpy="0 0 0"/>
+            <origin xyz="0 0 0" rpy="-1.57 0 0"/>
             <geometry>
                 <mesh filename="${mesh_location}/R_3_Wheel_Link.STL"/>
@@ -61,5 +61,5 @@
         </visual>
         <collision>
-            <origin xyz="0 0 0.035" rpy="0 0 0"/>
+            <origin xyz="0 0.035 0" rpy="-1.57 0 0"/>
             <geometry>
                 <cylinder radius="${wheel_radius}" length="${wheel_thickness}"/>
@@ -67,15 +67,10 @@
         </collision>
     </link>
-    <!-- Right Wheel 1 Joint -->
+    <!-- Right Wheel 3 Joint -->
     <joint name="R_3_Wheel_Joint" type="continuous">
-        <origin xyz="0.1542 -0.1266 -0.086" rpy="0 0 0"/>
+        <origin xyz="0.1542 -0.1266 -0.086" rpy=" 1.57 0 -3.14"/>
         <parent link="R_Boggie_Link"/>
         <child link="R_3_Wheel_Link"/>
-        <xacro:if value="$(arg invert_right_wheels)">
-            <axis xyz="0 0 -1"/>
-        </xacro:if>
-        <xacro:unless value="$(arg invert_right_wheels)">
-            <axis xyz="0 0 1"/>
-        </xacro:unless>
+        <axis xyz="0 1 0"/>
         <dynamics damping="0.01" friction="0.01"/>
     </joint>
@@ -83,5 +78,5 @@
     <link name="R_2_Wheel_Link">
         <inertial>
-            <origin xyz="0 0 0.0350608778434713" rpy="0 0 0"/>
+            <origin xyz="0 0.0350608778434713 0" rpy="-1.57 0 0"/>
             <mass value="${wheel_mass}"/>
             <inertia
@@ -94,5 +89,5 @@
         </inertial>
         <visual>
-            <origin xyz="0 0 0" rpy="0 0 0"/>
+            <origin xyz="0 0 0" rpy="-1.57 0 0"/>
             <geometry>
                 <mesh filename="${mesh_location}/R_2_Wheel_Link.STL"/>
@@ -101,5 +96,5 @@
         </visual>
         <collision>
-            <origin xyz="0 0 0.035" rpy="0 0 0"/>
+            <origin xyz="0 0.035 0" rpy="-1.57 0 0"/>
             <geometry>
                 <cylinder radius="${wheel_radius}" length="${wheel_thickness}"/>
@@ -109,19 +104,14 @@
     <!-- Right Wheel 2 Joint -->
     <joint name="R_2_Wheel_Joint" type="continuous">
-        <origin xyz="-0.1267 -0.1545 -0.086" rpy="0 0 0"/>
+        <origin xyz="-0.1267 -0.1545 -0.086" rpy=" 1.57 0 -3.14"/>
         <parent link="R_Boggie_Link"/>
         <child link="R_2_Wheel_Link"/>
-        <xacro:if value="$(arg invert_right_wheels)">
-            <axis xyz="0 0 -1"/>
-        </xacro:if>
-        <xacro:unless value="$(arg invert_right_wheels)">
-            <axis xyz="0 0 1"/>
-        </xacro:unless>
+        <axis xyz="0 1 0"/>
         <dynamics damping="0.01" friction="0.01"/>
     </joint>
-    <!-- Right Wheel 3 -->
+    <!-- Right Wheel 1 -->
     <link name="R_1_Wheel_Link">
         <inertial>
-            <origin xyz="0 0 0.0350608778434713" rpy="0 0 0"/>
+            <origin xyz="0 0.0350608778434713 0" rpy="-1.57 0 0"/>
             <mass value="${wheel_mass}"/>
             <inertia
@@ -134,5 +124,5 @@
         </inertial>
         <visual>
-            <origin xyz="0 0 0" rpy="0 0 0"/>
+            <origin xyz="0 0 0" rpy="-1.57 0 0"/>
             <geometry>
                 <mesh filename="${mesh_location}/R_1_Wheel_Link.STL"/>
@@ -141,5 +131,5 @@
         </visual>
         <collision>
-            <origin xyz="0 0 0.035" rpy="0 0 0"/>
+            <origin xyz="0 0.035 0" rpy="-1.57 0 0"/>
             <geometry>
                 <cylinder radius="${wheel_radius}" length="${wheel_thickness}"/>
@@ -149,13 +139,8 @@
     <!-- Right Wheel 3 Joint -->
     <joint name="R_1_Wheel_Joint" type="continuous">
-        <origin xyz="-0.276 -0.1541 -0.0760000000000001" rpy="0 0 0"/>
+        <origin xyz="-0.276 -0.1541 -0.0760000000000001" rpy=" 1.57 0 -3.14"/>
         <parent link="R_Rocker_Link"/>
         <child link="R_1_Wheel_Link"/>
-        <xacro:if value="$(arg invert_right_wheels)">
-            <axis xyz="0 0 -1"/>
-        </xacro:if>
-        <xacro:unless value="$(arg invert_right_wheels)">
-            <axis xyz="0 0 1"/>
-        </xacro:unless>
+        <axis xyz="0 1 0"/>
         <dynamics damping="0.01" friction="0.01"/>
     </joint>

File: rover_description/urdf/rover_control.xacro (robot description, xacro)
@@ -83,5 +83,7 @@
   <!-- ================================================================
        REAL HARDWARE  (ODrive S1 x6 via CAN bus)
-       Velocity limits: ±11.52 rad/s (110 RPM rated, r=0.110 m → ~1.27 m/s)
+       Velocity limits: ±25 rad/s (motor rated for 110 RPM / ~11.52 rad/s —
+                         raised past rating, confirm ODrive vel_limit and
+                         motor/gearbox can sustain this before running)
        Effort limits  : ±5 Nm (motor rated torque)
        ================================================================ -->
@@ -96,6 +98,6 @@
         <param name="node_id">3</param>
         <command_interface name="velocity">
-          <param name="min">-11.52</param>
-          <param name="max"> 11.52</param>
+          <param name="min">-50</param>
+          <param name="max"> 50</param>
         </command_interface>
         <command_interface name="effort">
@@ -110,6 +112,6 @@
         <param name="node_id">4</param>
         <command_interface name="velocity">
-          <param name="min">-11.52</param>
-          <param name="max"> 11.52</param>
+          <param name="min">-50</param>
+          <param name="max"> 50</param>
         </command_interface>
         <command_interface name="effort">
@@ -124,6 +126,6 @@
         <param name="node_id">5</param>
         <command_interface name="velocity">
-          <param name="min">-11.52</param>
-          <param name="max"> 11.52</param>
+          <param name="min">-50</param>
+          <param name="max"> 50</param>
         </command_interface>
         <command_interface name="effort">
@@ -139,6 +141,6 @@
         <param name="node_id">2</param>
         <command_interface name="velocity">
-          <param name="min">-11.52</param>
-          <param name="max"> 11.52</param>
+          <param name="min">-50</param>
+          <param name="max"> 50</param>
         </command_interface>
         <command_interface name="effort">
@@ -153,6 +155,6 @@
         <param name="node_id">1</param>
         <command_interface name="velocity">
-          <param name="min">-11.52</param>
-          <param name="max"> 11.52</param>
+          <param name="min">-50</param>
+          <param name="max"> 50</param>
         </command_interface>
         <command_interface name="effort">
@@ -167,6 +169,6 @@
         <param name="node_id">0</param>
         <command_interface name="velocity">
-          <param name="min">-11.52</param>
-          <param name="max"> 11.52</param>
+          <param name="min">-50</param>
+          <param name="max"> 50</param>
         </command_interface>
         <command_interface name="effort">
