Commit message: Add camera/IMU meshes, fold in ros_odrive, drop gz_ros2_control gitlink
Adds RealSense d435/ZED2i xacros and mesh, IMU data processing tweaks,
controller/teleop config updates, and rover description launch/urdf
fixes. ros_odrive is now tracked as regular files (previously an
untracked nested repo) so its ROS driver changes are included. The
__pycache__ artifact is ignored going forward.

File: rover_description/urdf/common_properties.xacro (robot description, xacro)
@@ -24,3 +24,5 @@
     <!-- Enable D435i -->
     <xacro:property name="enable_D435i" value="false"/>
+    <!-- Enable ZED 2i -->
+    <xacro:property name="enable_zed2i" value="true"/>
 </robot>

File: rover_description/urdf/my_robot.urdf.xacro (robot description, xacro)
@@ -13,3 +13,4 @@
     <xacro:include filename="right_link.xacro" />
     <xacro:include filename="rover_control.xacro" />
+    <xacro:include filename="zed2i.xacro"/>
 </robot>

File: rover_description/urdf/rover_control.xacro (robot description, xacro)
@@ -97,4 +97,5 @@
       <joint name="L_1_Wheel_Joint">
         <param name="node_id">3</param>
+        <param name="direction">1</param>
         <command_interface name="velocity">
           <param name="min">-50</param>
@@ -111,4 +112,5 @@
       <joint name="L_2_Wheel_Joint">
         <param name="node_id">4</param>
+        <param name="direction">1</param>
         <command_interface name="velocity">
           <param name="min">-50</param>
@@ -125,4 +127,5 @@
       <joint name="L_3_Wheel_Joint">
         <param name="node_id">5</param>
+        <param name="direction">1</param>
         <command_interface name="velocity">
           <param name="min">-50</param>
@@ -140,4 +143,5 @@
       <joint name="R_1_Wheel_Joint">
         <param name="node_id">2</param>
+        <param name="direction">-1</param>
         <command_interface name="velocity">
           <param name="min">-50</param>
@@ -154,4 +158,5 @@
       <joint name="R_2_Wheel_Joint">
         <param name="node_id">1</param>
+        <param name="direction">-1</param>
         <command_interface name="velocity">
           <param name="min">-50</param>
@@ -168,4 +173,5 @@
       <joint name="R_3_Wheel_Joint">
         <param name="node_id">0</param>
+        <param name="direction">-1</param>
         <command_interface name="velocity">
           <param name="min">-50</param>
