Commit message: Fix real-hardware controller pipeline and rgbd camera rename
Real robot: fix joystick deadman button (7 -> 5, matched to actual
gamepad), per-motor ODrive direction signs discovered via live testing,
and remap imu_restamp to /imu/data. Rename zed2i.xacro to
rgbd_camera.xacro with associated urdf/config/launch updates, plus
pointcloud display launch and mapping pipeline notes.

Co-Authored-By: Claude Sonnet 5 <noreply@anthropic.com>

File: rover_description/urdf/common_properties.xacro (robot description, xacro)
@@ -24,5 +24,5 @@
     <!-- Enable D435i -->
     <xacro:property name="enable_D435i" value="false"/>
-    <!-- Enable ZED 2i -->
-    <xacro:property name="enable_zed2i" value="true"/>
+    <!-- Enable RGB-D camera -->
+    <xacro:property name="enable_rgbd_camera" value="true"/>
 </robot>

File: rover_description/urdf/my_robot.urdf.xacro (robot description, xacro)
@@ -13,4 +13,4 @@
     <xacro:include filename="right_link.xacro" />
     <xacro:include filename="rover_control.xacro" />
-    <xacro:include filename="zed2i.xacro"/>
+    <xacro:include filename="rgbd_camera.xacro"/>
 </robot>

File: rover_description/urdf/rgbd_camera.xacro (robot description, xacro)
@@ -1,18 +1,37 @@
 <?xml version="1.0"?>
-<robot xmlns:xacro="http://www.ros.org/wiki/xacro" name="zed2i_camera">
-    <!-- Kinematic model (frames + mesh) comes from the official Stereolabs package -->
-    <xacro:include filename="$(find zed_description)/urdf/zed_macro.urdf.xacro" />
-    <!-- Mount point, reusing the same chassis location the D435i used -->
-    <joint name="zed_camera_mount_joint" type="fixed">
+<robot xmlns:xacro="http://www.ros.org/wiki/xacro" name="rgbd_camera">
+    <!-- Mount point on the chassis -->
+    <joint name="camera_mount_joint" type="fixed">
         <origin xyz="0.2756 0.0025 0.2535" rpy="0 0 0"/>
         <parent link="base_link"/>
-        <child link="zed_camera_link"/>
+        <child link="camera_center"/>
     </joint>
-    <xacro:zed_camera name="zed" model="zed2i">
-        <origin xyz="0 0 0" rpy="0 0 0"/>
-    </xacro:zed_camera>
+    <link name="camera_center">
+        <visual>
+            <geometry>
+                <box size="0.175 0.030 0.033"/>
+            </geometry>
+            <material name="gray"/>
+        </visual>
+        <collision>
+            <geometry>
+                <box size="0.175 0.030 0.033"/>
+            </geometry>
+        </collision>
+        <inertial>
+            <mass value="0.166"/>
+            <inertia ixx="1e-5" ixy="0" ixz="0" iyy="1e-5" iyz="0" izz="1e-5"/>
+        </inertial>
+    </link>
+    <!-- Optical frame follows the ROS camera convention (x-right, y-down, z-forward) -->
+    <joint name="left_camera_optical_joint" type="fixed">
+        <origin xyz="0 0 0" rpy="${-PI/2} 0 ${-PI/2}"/>
+        <parent link="camera_center"/>
+        <child link="left_camera_frame_optical"/>
+    </joint>
+    <link name="left_camera_frame_optical"/>
     <!-- Gazebo configuration for Ionic/ROS2 Jazzy -->
-    <xacro:if value="${enable_zed2i}">
-        <gazebo reference="zed_camera_center">
+    <xacro:if value="${enable_rgbd_camera}">
+        <gazebo reference="camera_center">
             <self_collide>0</self_collide>
             <enable_wind>0</enable_wind>
@@ -23,6 +42,6 @@
             <kd>1</kd>
             <!-- Left color camera - 15 Hz, matching the rest of the rig's render budget -->
-            <sensor name="zed_left_color" type="camera">
-                <camera name="zed_left">
+            <sensor name="camera_left_color" type="camera">
+                <camera name="camera_left">
                     <horizontal_fov>1.8</horizontal_fov>
                     <image>
@@ -44,10 +63,10 @@
                 <update_rate>15</update_rate>
                 <visualize>false</visualize>
-                <topic>zed/left/image_rect_color</topic>
-                <gz_frame_id>zed_left_camera_frame_optical</gz_frame_id>
+                <topic>camera/left/image_rect_color</topic>
+                <gz_frame_id>left_camera_frame_optical</gz_frame_id>
             </sensor>
-            <!-- Depth, registered to the left camera per ZED SDK convention -->
-            <sensor name="zed_depth" type="depth_camera">
-                <camera name="zed_depth">
+            <!-- Depth, registered to the left camera -->
+            <sensor name="camera_depth" type="depth_camera">
+                <camera name="camera_depth">
                     <horizontal_fov>1.8</horizontal_fov>
                     <image>
@@ -69,6 +88,6 @@
                 <update_rate>15</update_rate>
                 <visualize>false</visualize>
-                <topic>zed/depth/depth_registered</topic>
-                <gz_frame_id>zed_left_camera_frame_optical</gz_frame_id>
+                <topic>camera/depth/depth_registered</topic>
+                <gz_frame_id>left_camera_frame_optical</gz_frame_id>
             </sensor>
         </gazebo>

File: rover_description/urdf/rover_control.xacro (robot description, xacro)
@@ -87,4 +87,10 @@
                          motor/gearbox can sustain this before running)
        Effort limits  : ±5 Nm (motor rated torque)
+       CAN node_id -> wheel location (confirmed against physical rover;
+       direction signs below were tuned per-motor, not per-position — they
+       do NOT follow a left/right or front/bogie pattern):
+         node_id 3 -> L_1 (front left)     node_id 2 -> R_1 (front right)
+         node_id 4 -> L_2 (middle left)    node_id 1 -> R_2 (middle right)
+         node_id 5 -> L_3 (rear left)      node_id 0 -> R_3 (rear right)
        ================================================================ -->
   <xacro:unless value="$(arg use_sim)">
@@ -95,7 +101,7 @@
       </hardware>
       <!-- LEFT WHEELS -->
-      <joint name="L_1_Wheel_Joint">
+      <joint name="L_1_Wheel_Joint"> <!-- front left -->
         <param name="node_id">3</param>
-        <param name="direction">1</param>
+        <param name="direction">-1</param>
         <command_interface name="velocity">
           <param name="min">-50</param>
@@ -110,7 +116,7 @@
         <state_interface name="effort"/>
       </joint>
-      <joint name="L_2_Wheel_Joint">
+      <joint name="L_2_Wheel_Joint"> <!-- middle left -->
         <param name="node_id">4</param>
-        <param name="direction">1</param>
+        <param name="direction">-1</param>
         <command_interface name="velocity">
           <param name="min">-50</param>
@@ -125,5 +131,5 @@
         <state_interface name="effort"/>
       </joint>
-      <joint name="L_3_Wheel_Joint">
+      <joint name="L_3_Wheel_Joint"> <!-- rear left -->
         <param name="node_id">5</param>
         <param name="direction">1</param>
@@ -141,7 +147,7 @@
       </joint>
       <!-- RIGHT WHEELS -->
-      <joint name="R_1_Wheel_Joint">
+      <joint name="R_1_Wheel_Joint"> <!-- front right -->
         <param name="node_id">2</param>
-        <param name="direction">-1</param>
+        <param name="direction">1</param>
         <command_interface name="velocity">
           <param name="min">-50</param>
@@ -156,7 +162,7 @@
         <state_interface name="effort"/>
       </joint>
-      <joint name="R_2_Wheel_Joint">
+      <joint name="R_2_Wheel_Joint"> <!-- middle right -->
         <param name="node_id">1</param>
-        <param name="direction">-1</param>
+        <param name="direction">1</param>
         <command_interface name="velocity">
           <param name="min">-50</param>
@@ -171,5 +177,5 @@
         <state_interface name="effort"/>
       </joint>
-      <joint name="R_3_Wheel_Joint">
+      <joint name="R_3_Wheel_Joint"> <!-- rear right -->
         <param name="node_id">0</param>
         <param name="direction">-1</param>
