Commit message: Add NDT scan-matching localization and sim lidar/IMU mapping updates
- navigation: ndt_localize.launch.py runs Autoware ndt_scan_matcher against a
  PCD map, with ndt_ekf_bridge.py feeding it a pose guess and a map-frame EKF
  (ekf_map.yaml) fusing the NDT pose to publish map -> odom
- navigation: mesh_to_pcd.py samples the Gazebo terrain mesh into
  terrain_world.pcd; RTAB-Map lidar mapping gets an IMU gravity constraint
- ekf: 3D mode with absolute IMU roll/pitch/yaw; drop imu_restamp for sim-only
- rover_description: lidar.xacro, marsyard2026 world, RViz launched from
  my_robot.launch.py on the NVIDIA GPU, gazebo bridge and URDF updates
- ignore large generated data (point clouds, terrain meshes) from git

Co-Authored-By: Claude Sonnet 5.5 <noreply@anthropic.com>

File: rover_description/urdf/aries_gazebo.xacro (robot description, xacro)
@@ -131,6 +131,4 @@
     <maxVel>0.1</maxVel>
     <fdir1>1 0 0</fdir1>
-  </gazebo>
-  <gazebo reference="Lidar_Link">
   </gazebo>
   <!-- Gazebo Plugin for Joint State Publisher -->
@@ -285,13 +283,77 @@
         </plugin>
   </gazebo>
-  <gazebo reference="imu_frame">
-      <sensor name="imu_sensor" type="imu">
-          <always_on>1</always_on>
-          <update_rate>100</update_rate>
-          <gz_frame_id>imu_frame</gz_frame_id>
-          <visualize>true</visualize>
-          <topic>/imu</topic>
-      </sensor>
-  </gazebo>
+<gazebo reference="imu_frame">
+    <sensor name="imu_sensor" type="imu">
+        <always_on>1</always_on>
+        <update_rate>100</update_rate>
+        <gz_frame_id>imu_frame</gz_frame_id>
+        <visualize>true</visualize>
+        <topic>/imu</topic>
+        <imu>
+            <!-- Gyroscope noise, rad/s (MPU6050-like, after calibration) -->
+            <angular_velocity>
+                <x>
+                    <noise type="gaussian">
+                        <mean>0.0</mean>
+                        <stddev>0.0009</stddev>
+                        <bias_mean>0.0005</bias_mean>
+                        <bias_stddev>0.0001</bias_stddev>
+                        <dynamic_bias_stddev>0.00002</dynamic_bias_stddev>
+                        <dynamic_bias_correlation_time>400.0</dynamic_bias_correlation_time>
+                    </noise>
+                </x>
+                <y> <noise type="gaussian">
+                        <mean>0.0</mean>
+                        <stddev>0.0009</stddev>
+                        <bias_mean>0.0005</bias_mean>
+                        <bias_stddev>0.0001</bias_stddev>
+                        <dynamic_bias_stddev>0.00002</dynamic_bias_stddev>
+                        <dynamic_bias_correlation_time>400.0</dynamic_bias_correlation_time>
+                    </noise>
+                </y>
+                <z> <noise type="gaussian">
+                        <mean>0.0</mean>
+                        <stddev>0.0009</stddev>
+                        <bias_mean>0.0005</bias_mean>
+                        <bias_stddev>0.0001</bias_stddev>
+                        <dynamic_bias_stddev>0.00002</dynamic_bias_stddev>
+                        <dynamic_bias_correlation_time>400.0</dynamic_bias_correlation_time>
+                    </noise>
+                </z>
+            </angular_velocity>
+            <!-- Accelerometer noise, m/s² (MPU6050-like, after calibration) -->
+            <linear_acceleration>
+                <x>
+                    <noise type="gaussian">
+                        <mean>0.0</mean>
+                        <stddev>0.04</stddev>
+                        <bias_mean>0.05</bias_mean>
+                        <bias_stddev>0.01</bias_stddev>
+                        <dynamic_bias_stddev>0.002</dynamic_bias_stddev>
+                        <dynamic_bias_correlation_time>300.0</dynamic_bias_correlation_time>
+                    </noise>
+                </x>
+                <y> <noise type="gaussian">
+                        <mean>0.0</mean>
+                        <stddev>0.04</stddev>
+                        <bias_mean>0.05</bias_mean>
+                        <bias_stddev>0.01</bias_stddev>
+                        <dynamic_bias_stddev>0.002</dynamic_bias_stddev>
+                        <dynamic_bias_correlation_time>300.0</dynamic_bias_correlation_time>
+                    </noise>
+                 </y>
+                <z> <noise type="gaussian">
+                        <mean>0.0</mean>
+                        <stddev>0.04</stddev>
+                        <bias_mean>0.05</bias_mean>
+                        <bias_stddev>0.01</bias_stddev>
+                        <dynamic_bias_stddev>0.002</dynamic_bias_stddev>
+                        <dynamic_bias_correlation_time>300.0</dynamic_bias_correlation_time>
+                    </noise>
+                </z>
+            </linear_acceleration>
+        </imu>
+    </sensor>
+</gazebo>
   <!-- Gazebo Plugin for Diff Drive (disabled when ros2_control handles driving) -->
   <xacro:unless value="$(arg use_sim)">

File: rover_description/urdf/common_properties.xacro (robot description, xacro)
@@ -23,6 +23,6 @@
     <xacro:property name="enable_lidar" value="false"/>
     <!-- Enable D435i -->
-    <xacro:property name="enable_D435i" value="false"/>
+    <xacro:property name="enable_D435i" value="true"/>
     <!-- Enable RGB-D camera -->
-    <xacro:property name="enable_rgbd_camera" value="true"/>
+    <xacro:property name="enable_rgbd_camera" value="false"/>
 </robot>

File: rover_description/urdf/my_robot.urdf.xacro (robot description, xacro)
@@ -13,4 +13,6 @@
     <xacro:include filename="right_link.xacro" />
     <xacro:include filename="rover_control.xacro" />
-    <xacro:include filename="rgbd_camera.xacro"/>
+    <!-- D435i disabled for now (lidar only) -->
+    <!-- <xacro:include filename="d435i.xacro"/> -->
+    <xacro:include filename="lidar.xacro"/>
 </robot>
